Commit message: Perfect merge for scan

File: turtlebot3_simulations/turtlebot3_gazebo/urdf/turtlebot3_waffle.urdf (robot description, URDF)
Before this commit: robot turtlebot3_waffle_pi, 13 links, 12 joints
Links:
- removed link base_scan_rear
- added link base_scan_back, mass 0.114; collision cylinder length=0.0315 radius=0.055; visual mesh filename=package://turtlebot3_description/meshes/sensors/lds.stl scale=0.001 0.001 0.001
Joints:
- joint scan_rear_joint: child base_scan_rear -> base_scan_back
