Commit message: Revise the urdf adding Ultrasonic & test complete

File: turtlebot3/turtlebot3_description/urdf/turtlebot3_waffle.urdf (robot description, URDF)
Before this commit: robot turtlebot3_waffle, 15 links, 14 joints
Links:
- removed link camera_depth_frame
- removed link camera_depth_optical_frame
- removed link laser_front
- removed link laser_rear
- added link base_scan_front, mass 0.114; collision cylinder length=0.0315 radius=0.055; visual mesh filename=package://turtlebot3_description/meshes/sensors/lds.stl scale=0.001 0.001 0.001
- added link base_scan_rear, mass 0.114; collision cylinder length=0.0315 radius=0.055; visual mesh filename=package://turtlebot3_description/meshes/sensors/lds.stl scale=0.001 0.001 0.001
- added link ultrasonic_front; visual box size=0.03 0.06 0.02
- added link ultrasonic_left; visual box size=0.03 0.06 0.02
- added link ultrasonic_right; visual box size=0.03 0.06 0.02
- link base_link: geometry collision box size=0.266 0.266 0.094; visual mesh filename=package://turtlebot3_description/meshes/bases/waffle_pi_bas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 scale=0.001 0.001 0.001
- link camera_link: geometry collision box size=0.015 0.030 0.027
Joints:
- removed joint camera_depth_joint
- removed joint camera_depth_optical_joint
- added joint ultrasonic_front_joint: type fixed, parent base_link, child ultrasonic_front, origin xyz=0.064 0 0.094 rpy=0 0 0
- added joint ultrasonic_left_joint: type fixed, parent base_link, child ultrasonic_left, origin xyz=0.064 0.135 0.094 rpy=0 0 0.785
- added joint ultrasonic_right_joint: type fixed, parent base_link, child ultrasonic_right, origin xyz=0.064 -0.135 0.094 rpy=0 0 -0.785
- joint camera_joint: origin xyz=0.064 -0.065 0.094 rpy=0 0 0 -> xyz=0.073 -0.011 0.084 rpy=0 0 0
- joint camera_rgb_joint: origin xyz=0.005 0.018 0.013 rpy=0 0 0 -> xyz=0.003 0.011 0.009 rpy=0 0 0
- joint scan_front_joint: child laser_front -> base_scan_front; origin xyz=0.536 0 0.122 rpy=0 0 0 -> xyz=0.05 0 0 rpy=0 0 0
- joint scan_rear_joint: child laser_rear -> base_scan_rear; origin xyz=-0.664 0 0.122 rpy=0 0 -3.141592 -> xyz=-0.05 0 0 rpy=0 0 3.141592

Commit message: Update

File: turtlebot3/turtlebot3_description/urdf/turtlebot3_waffle.urdf (robot description, URDF)
Before this commit: robot turtlebot3_waffle, 15 links, 14 joints
Joints:
- joint camera_joint: origin xyz=0.064 -0.065 0.094 rpy=0 0 0 -> xyz=0.064 0.0 0.094 rpy=0 0 0

File: turtlebot3_simulations/turtlebot3_gazebo/urdf/turtlebot3_waffle.urdf (robot description, URDF)
Before this commit: robot turtlebot3_waffle_pi, 13 links, 12 joints
Links:
- added link camera_rear_link
- added link camera_rear_rgb_frame
- added link camera_rear_rgb_optical_frame
- link camera_link: geometry 
Joints:
- added joint camera_rear_joint: type fixed, parent base_link, child camera_rear_link, origin xyz=-0.190 0.0 0.094 rpy=0 0 0
- added joint camera_rear_rgb_joint: type fixed, parent camera_rear_link, child camera_rear_rgb_frame, origin xyz=0.0 0.0 0.0 rpy=0 0 3.14
- added joint camera_rear_rgb_optical_joint: type fixed, parent camera_rear_rgb_frame, child camera_rear_rgb_optical_frame, origin xyz=0 0 0 rpy=-1.57 0 -1.57
- joint camera_joint: origin xyz=0.073 -0.011 0.084 rpy=0 0 0 -> xyz=0.064 0.0 0.094 rpy=0 0 0
- joint camera_rgb_joint: origin xyz=0.003 0.011 0.009 rpy=0 0 0 -> xyz=0.0 0.0 0.0 rpy=0 0 0
- joint scan_front_joint: origin xyz=0.05 0 0 rpy=0 0 0 -> xyz=0.0 0 0 rpy=0 0 0
- joint scan_joint: origin xyz=-0.064 0 0.122 rpy=0 0 0 -> xyz=0.0 0 0.122 rpy=0 0 0
- joint scan_rear_joint: origin xyz=-0.05 0 0 rpy=0 0 3.141592 -> xyz=-0.1 0 0 rpy=0 0 3.141592
